Commit message: wip

File: urdf/RGBD_camera_bot.xacro (robot description, xacro)
@@ -1,4 +1,4 @@
 <?xml version='1.0'?>
-<robot name="slam_project" xmlns:xacro="http://www.ros.org/wiki/xacro">
+<robot name="RGBD_camera_bot" xmlns:xacro="http://www.ros.org/wiki/xacro">
   <!-- source: https://github.com/tu-darmstadt-ros-pkg/hector_models/blob/indigo-devel/hector_xacro_tools/urdf/inertia_tensors.urdf.xacro -->
   <xacro:include filename="$(find slam_project)/urdf/inertia_tensors.urdf.xacro" />
@@ -11,5 +11,5 @@
   </joint>
   <joint type="continuous" name="left_wheel_hinge">
-    <origin xyz="0 0.23 -0.26" rpy="0 0 0"/>
+    <origin xyz="0 0.15 0" rpy="0 0 0"/>
     <child link="left_wheel"/>
     <parent link="chassis"/>
@@ -19,5 +19,5 @@
   </joint>
   <joint type="continuous" name="right_wheel_hinge">
-    <origin xyz="0 -0.23 -0.26" rpy="0 0 0"/>
+    <origin xyz="0 -0.15 0" rpy="0 0 0"/>
     <child link="right_wheel"/>
     <parent link="chassis"/>
@@ -27,5 +27,5 @@
   </joint>
   <joint type="fixed" name="camera_joint">
-    <origin xyz="0.2 0 .2" rpy="0 0 0"/>
+    <origin xyz="0.2 0 0" rpy="0 0 0"/>
     <child link="camera"/>
     <parent link="chassis"/>
@@ -35,5 +35,5 @@
   </joint>
   <joint type="fixed" name="hokuyo_joint">
-    <origin xyz="0 0 0.335" rpy="0 0 0"/>
+    <origin xyz="0.15 0 0.08" rpy="0 0 0"/>
     <child link="hokuyo"/>
     <parent link="chassis"/>
@@ -43,5 +43,5 @@
   </joint>
   <joint type="fixed" name="front_caster_joint">
-    <origin xyz="0.15 0 -0.31" rpy="0 0 0"/>
+    <origin xyz="0.15 0 -0.05" rpy="0 0 0"/>
     <child link="front_caster"/>
     <parent link="chassis"/>
@@ -51,5 +51,5 @@
   </joint>
   <joint type="fixed" name="back_caster_joint">
-    <origin xyz="-0.15 0 -0.31" rpy="0 0 0"/>
+    <origin xyz="-0.15 0 -0.05" rpy="0 0 0"/>
     <child link="back_caster"/>
     <parent link="chassis"/>
@@ -146,11 +146,11 @@
   <link name='chassis'>
     <pose>0 0 0.1 0 0 0</pose>
-    <xacro:inertial_cylinder_with_pose mass="30.0" radius="0.2" z_length="0.6" >
+    <xacro:inertial_cuboid_with_pose mass="15.0" x_length=".4" y_length="0.2" z_length="0.1" >
       <origin xyz="0.0 0 0" rpy=" 0 0 0"/>
-    </xacro:inertial_cylinder_with_pose>
+    </xacro:inertial_cuboid_with_pose>
     <collision name='collision'>
       <origin xyz="0 0 0" rpy=" 0 0 0"/>
       <geometry>
-        <cylinder length="0.6" radius="0.2"/>
+        <box size=".4 .2 .1"/>
       </geometry>
     </collision>
@@ -158,5 +158,5 @@
       <origin xyz="0 0 0" rpy=" 0 0 0"/>
       <geometry>
-        <cylinder length="0.6" radius="0.2"/>
+        <box size=".4 .2 .1"/>
       </geometry>
     </visual>

Commit message: camera processed, points point in wrong direction

File: urdf/RGBD_camera_bot.xacro (robot description, xacro)
@@ -28,5 +28,5 @@
   <joint type="fixed" name="camera_joint">
     <origin xyz="0.2 0 0" rpy="0 0 0"/>
-    <child link="camera"/>
+    <child link="camera_rgbd_frame"/>
     <parent link="chassis"/>
     <axis xyz="0 1 0" rpy="0 0 0"/>
@@ -104,5 +104,5 @@
     </visual>
   </link>
-  <link name='camera'>
+  <link name='camera_rgbd_frame'>
       <xacro:inertial_cuboid_with_pose mass=".1" x_length="0.05" y_length="0.05" z_length="0.05" >
         <origin xyz="0.0 0 0" rpy=" 0 0 0"/>
